Commit message: adding camera tutorials

File: ornithopter/urdf/ornithopter.urdf.xacro (robot description, xacro)
@@ -5,5 +5,5 @@
     <inertial>
       <origin xyz="0 0.03 0" rpy="0 0 0"/>
-      <mass value="0.00002"/>
+      <mass value="0.2"/>
       <inertia ixx="0.01" ixy="0.0" ixz="0.0" iyy="0.001" iyz="0.0" izz="0.001"/>
     </inertial>
@@ -31,5 +31,5 @@
     <inertial>
       <origin xyz="0 0 0.0" rpy="0 0 0"/>
-      <mass value="0.0001"/>
+      <mass value="0.9"/>
       <inertia ixx="0.05" ixy="0.0" ixz="0.0" iyy="0.08" iyz="0.0" izz="0.08"/>
     </inertial>
@@ -49,5 +49,5 @@
     <inertial>
       <origin xyz="0 0 0" rpy="0 0 0"/>
-      <mass value="0.000004"/>
+      <mass value="0.4"/>
       <inertia ixx="0.005" ixy="0.0" ixz="0.0" iyy="0.001" iyz="0.0" izz="0.001"/>
     </inertial>
@@ -87,5 +87,5 @@
     <inertial>
       <origin xyz="0 0 0" rpy="0 0 0"/>
-      <mass value="0.000004"/>
+      <mass value="0.4"/>
       <inertia ixx="0.005" ixy="0.0" ixz="0.0" iyy="0.001" iyz="0.0" izz="0.001"/>
     </inertial>
@@ -126,5 +126,5 @@
     <inertial>
       <origin xyz="0 0 0" rpy="0 0 0"/>
-      <mass value="0.00004"/>
+      <mass value="0.4"/>
       <inertia ixx="0.005" ixy="0.0" ixz="0.0" iyy="0.005" iyz="0.0" izz="0.005"/>
     </inertial>
@@ -151,5 +151,5 @@
     <inertial>
       <origin xyz="0 0 0" rpy="0 0 0"/>
-      <mass value="0.00004"/>
+      <mass value="0.4"/>
       <inertia ixx="0.005" ixy="0.0" ixz="0.0" iyy="0.005" iyz="0.0" izz="0.005"/>
     </inertial>
@@ -226,9 +226,9 @@
       <link_name>link_4</link_name>
       <!--direction-->
-      <forward>0 0 1</forward>
-      <upward>0 0 0</upward>
+      <forward>1 0 0</forward>
+      <upward>0 1 0</upward>
       <cp>0 0.05 -0.16</cp>
       <!-- geometry -->
-      <area>0.25</area>
+      <area>0.000000105</area>
       <fluid_density>1.225</fluid_density>
       <!-- aerodynamic coefficients -->
@@ -245,9 +245,9 @@
       <link_name>link_6</link_name>
       <!--direction-->
-      <forward>0 0 1</forward>
+      <forward>1 0 0</forward>
       <upward>0 1 0</upward>
       <cp>-0.12 0 0.12</cp>
       <!-- geometry -->
-      <area>0.25</area>
+      <area>0.000000105</area>
       <fluid_density>1.225</fluid_density>
       <!-- aerodynamic coefficients -->
